File: board/bootflash.kicad_sch (KiCad schematic)
At the start: 0 parts

Commit message: Finished initial schematic, ready for signoff review
Parts:
- added C182: 4.7 uF, azonenberg_pcb:EIA_0603_CAP_NOSILK, symbol device:C
- added C183, C184: 0.47 uF, azonenberg_pcb:EIA_0402_CAP_NOSILK, symbol device:C
- added R131, R132, R133, R134: 33, azonenberg_pcb:EIA_0402_RES_NOSILK, symbol device:R
- added U14: S25FLxxxS_BGA24_5x5_VIO, azonenberg_pcb:BGA_24_6x8_DEPOP1_1MM, symbol memory-azonenberg:S25FLxxxS_BGA24_5x5_VIO
Connections:
- net 3V3: now also C182.1, C183.1, C184.1, U14.A4 (RESET_N), U14.B4 (VDD), U14.E4 (VIO)
- net FLASH_CS_N: now also U14.C2 (CS_N)
- net FLASH_DQ0: now also R131.2
- net FLASH_DQ1: now also R132.2
- net FLASH_DQ2: now also R133.2
- net FLASH_DQ3: now also R134.2
- net FLASH_SCK: now also U14.B2 (SCK)
- net GND: now also C182.2, C183.2, C184.2, U14.B3 (VSS)
- new net: R134.1, U14.D4 (RESET_N/DQ3)
- new net: R133.1, U14.C4 (WP_N/DQ2)
- new net: R132.1, U14.D2 (MISO/DQ1)
- new net: R131.1, U14.D3 (MOSI/DQ0)
Changed lines of the file:
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@@
     (comment 1 "Andrew D. Zonenberg")
   )
-  (hierarchical_label "FLASH_DQ1" (shape bidirectional) (at 125.73 60.96 0)
+  (junction (at 76.2 76.2) (diameter 0) (color 0 0 0 0)
+  )
+  (junction (at 76.2 83.82) (diameter 0) (color 0 0 0 0)
+  )
+  (wire (pts (xy 107.95 50.8) (xy 113.03 50.8))
+    (stroke (width 0) (type default) (color 0 0 0 0))
+  )
+  (wire (pts (xy 63.5 83.82) (xy 76.2 83.82))
+    (stroke (width 0) (type default) (color 0 0 0 0))
+  )
+  (wire (pts (xy 76.2 76.2) (xy 90.17 76.2))
+    (stroke (width 0) (type default) (color 0 0 0 0))
+  )
+  (wire (pts (xy 107.95 58.42) (xy 113.03 58.42))
+    (stroke (width 0) (type default) (color 0 0 0 0))
+  )
+  (wire (pts (xy 107.95 53.34) (xy 113.03 53.34))
+    (stroke (width 0) (type default) (color 0 0 0 0))
+  )
+  (wire (pts (xy 63.5 45.72) (xy 63.5 48.26))
+    (stroke (width 0) (type default) (color 0 0 0 0))
+  )
+  (wire (pts (xy 63.5 76.2) (xy 76.2 76.2))
+    (stroke (width 0) (type default) (color 0 0 0 0))
+  )
+  (wire (pts (xy 107.95 55.88) (xy 113.03 55.88))
+    (stroke (width 0) (type default) (color 0 0 0 0))
+  )
+  (wire (pts (xy 76.2 83.82) (xy 90.17 83.82))
+    (stroke (width 0) (type default) (color 0 0 0 0))
+  )
+  (label "3V3" (at 63.5 55.88 180)
+    (effects (font (size 1.27 1.27)) (justify right bottom))
+  )
+  (label "3V3" (at 63.5 76.2 180)
+    (effects (font (size 1.27 1.27)) (justify right bottom))
+  )
+  (label "GND" (at 63.5 83.82 180)
+    (effects (font (size 1.27 1.27)) (justify right bottom))
+  )
+  (hierarchical_label "FLASH_DQ1" (shape bidirectional) (at 113.03 53.34 0)
     (effects (font (size 1.27 1.27)) (justify left))
   )
-  (hierarchical_label "FLASH_SCK" (shape input) (at 124.46 46.99 0)
+  (hierarchical_label "FLASH_SCK" (shape input) (at 63.5 63.5 180)
+    (effects (font (size 1.27 1.27)) (justify right))
+  )
+  (hierarchical_label "FLASH_DQ2" (shape bidirectional) (at 113.03 55.88 0)
     (effects (font (size 1.27 1.27)) (justify left))
   )
-  (hierarchical_label "FLASH_DQ2" (shape bidirectional) (at 125.73 63.5 0)
+  (hierarchical_label "FLASH_DQ0" (shape bidirectional) (at 113.03 50.8 0)
     (effects (font (size 1.27 1.27)) (justify left))
   )
-  (hierarchical_label "FLASH_DQ0" (shape bidirectional) (at 125.73 58.42 0)
+  (hierarchical_label "GND" (shape input) (at 63.5 50.8 180)
+    (effects (font (size 1.27 1.27)) (justify right))
+  )
+  (hierarchical_label "FLASH_DQ3" (shape bidirectional) (at 113.03 58.42 0)
     (effects (font (size 1.27 1.27)) (justify left))
   )
-  (hierarchical_label "GND" (shape input) (at 138.43 25.4 0)
-    (effects (font (size 1.27 1.27)) (justify left))
+  (hierarchical_label "FLASH_CS_N" (shape input) (at 63.5 60.96 180)
+    (effects (font (size 1.27 1.27)) (justify right))
   )
-  (hierarchical_label "FLASH_DQ3" (shape bidirectional) (at 125.73 66.04 0)
-    (effects (font (size 1.27 1.27)) (justify left))
+  (hierarchical_label "3V3" (shape input) (at 63.5 45.72 180)
+    (effects (font (size 1.27 1.27)) (justify right))
   )
-  (hierarchical_label "FLASH_CS_N" (shape input) (at 124.46 35.56 0)
-    (effects (font (size 1.27 1.27)) (justify left))
+  (symbol (lib_id "device:R") (at 104.14 58.42 90) (unit 1)
+    (in_bom yes) (on_board yes)
+    (property "Reference" "R134" (id 0) (at 107.95 57.15 90))
+    (property "Value" "33" (id 1) (at 104.14 58.42 90))
+    (property "Footprint" "azonenberg_pcb:EIA_0402_RES_NOSILK" (id 2) (at 104.14 60.198 90)
+      (effects (font (size 1.27 1.27)) hide)
+    )
+    (property "Datasheet" "" (id 3) (at 104.14 58.42 0)
+      (effects (font (size 1.27 1.27)) hide)
+    )
+    (pin "1")
+    (pin "2")
   )
-  (hierarchical_label "3V3" (shape input) (at 121.92 26.67 0)
-    (effects (font (size 1.27 1.27)) (justify left))
+  (symbol (lib_id "memory-azonenberg:S25FLxxxS_BGA24_5x5_VIO") (at 68.58 64.77 0) (unit 1)
+    (in_bom yes) (on_board yes) (fields_autoplaced)
+    (property "Reference" "U14" (id 0) (at 81.915 40.0461 0)
+      (effects (font (size 1.524 1.524)))
+    )
+    (property "Value" "S25FLxxxS_BGA24_5x5_VIO" (id 1) (at 81.915 43.3251 0)
+      (effects (font (size 1.524 1.524)))
+    )
+    (property "Footprint" "azonenberg_pcb:BGA_24_6x8_DEPOP1_1MM" (id 2) (at 68.58 64.77 0)
+      (effects (font (size 1.524 1.524)) hide)
+    )
+    (property "Datasheet" "" (id 3) (at 68.58 64.77 0)
+      (effects (font (size 1.524 1.524)) hide)
+    )
+    (pin "A4")
+    (pin "B2")
+    (pin "B3")
+    (pin "B4")
+    (pin "C2")
+    (pin "C4")
+    (pin "D2")
+    (pin "D3")
+    (pin "D4")
+    (pin "E4")
+  )
+  (symbol (lib_id "device:C") (at 90.17 80.01 0) (unit 1)
+    (in_bom yes) (on_board yes)
+    (property "Reference" "C184" (id 0) (at 93.091 78.8416 0)
+      (effects (font (size 1.27 1.27)) (justify left))
+    )
+    (property "Value" "0.47 uF" (id 1) (at 93.091 81.153 0)
+      (effects (font (size 1.27 1.27)) (justify left))
+    )
+    (property "Footprint" "azonenberg_pcb:EIA_0402_CAP_NOSILK" (id 2) (at 91.1352 83.82 0)
+      (effects (font (size 1.27 1.27)) hide)
+    )
+    (property "Datasheet" "" (id 3) (at 90.17 80.01 0)
+      (effects (font (size 1.27 1.27)) hide)
+    )
+    (pin "1")
+    (pin "2")
+  )
+  (symbol (lib_id "device:C") (at 76.2 80.01 0) (unit 1)
+    (in_bom yes) (on_board yes)
+    (property "Reference" "C183" (id 0) (at 79.121 78.8416 0)
+      (effects (font (size 1.27 1.27)) (justify left))
+    )
+    (property "Value" "0.47 uF" (id 1) (at 79.121 81.153 0)
+      (effects (font (size 1.27 1.27)) (justify left))
+    )
+    (property "Footprint" "azonenberg_pcb:EIA_0402_CAP_NOSILK" (id 2) (at 77.1652 83.82 0)
+      (effects (font (size 1.27 1.27)) hide)
+    )
+    (property "Datasheet" "" (id 3) (at 76.2 80.01 0)
+      (effects (font (size 1.27 1.27)) hide)
+    )
+    (pin "1")
+    (pin "2")
+  )
+  (symbol (lib_id "device:R") (at 104.14 50.8 90) (unit 1)
+    (in_bom yes) (on_board yes)
+    (property "Reference" "R131" (id 0) (at 107.95 49.53 90))
+    (property "Value" "33" (id 1) (at 104.14 50.8 90))
+    (property "Footprint" "azonenberg_pcb:EIA_0402_RES_NOSILK" (id 2) (at 104.14 52.578 90)
+      (effects (font (size 1.27 1.27)) hide)
+    )
+    (property "Datasheet" "" (id 3) (at 104.14 50.8 0)
+      (effects (font (size 1.27 1.27)) hide)
+    )
+    (pin "1")
+    (pin "2")
+  )
+  (symbol (lib_id "device:C") (at 63.5 80.01 0) (unit 1)
+    (in_bom yes) (on_board yes)
+    (property "Reference" "C182" (id 0) (at 66.421 78.8416 0)
+      (effects (font (size 1.27 1.27)) (justify left))
+    )
+    (property "Value" "4.7 uF" (id 1) (at 66.421 81.153 0)
+      (effects (font (size 1.27 1.27)) (justify left))
+    )
+    (property "Footprint" "azonenberg_pcb:EIA_0603_CAP_NOSILK" (id 2) (at 64.4652 83.82 0)
+      (effects (font (size 1.27 1.27)) hide)
+    )
+    (property "Datasheet" "" (id 3) (at 63.5 80.01 0)
+      (effects (font (size 1.27 1.27)) hide)
+    )
+    (pin "1")
+    (pin "2")
+  )
+  (symbol (lib_id "device:R") (at 104.14 55.88 90) (unit 1)
+    (in_bom yes) (on_board yes)
+    (property "Reference" "R133" (id 0) (at 107.95 54.61 90))
+    (property "Value" "33" (id 1) (at 104.14 55.88 90))
+    (property "Footprint" "azonenberg_pcb:EIA_0402_RES_NOSILK" (id 2) (at 104.14 57.658 90)
+      (effects (font (size 1.27 1.27)) hide)
+    )
+    (property "Datasheet" "" (id 3) (at 104.14 55.88 0)
+      (effects (font (size 1.27 1.27)) hide)
+    )
+    (pin "1")
+    (pin "2")
+  )
+  (symbol (lib_id "device:R") (at 104.14 53.34 90) (unit 1)
+    (in_bom yes) (on_board yes)
+    (property "Reference" "R132" (id 0) (at 107.95 52.07 90))
+    (property "Value" "33" (id 1) (at 104.14 53.34 90))
+    (property "Footprint" "azonenberg_pcb:EIA_0402_RES_NOSILK" (id 2) (at 104.14 55.118 90)
+      (effects (font (size 1.27 1.27)) hide)
+    )
+    (property "Datasheet" "" (id 3) (at 104.14 53.34 0)
+      (effects (font (size 1.27 1.27)) hide)
+    )
+    (pin "1")
+    (pin "2")
   )
 )
