File: board/monpath.kicad_sch (KiCad schematic)
At the start: 1 part, among them U4 XC7S15-1FTGB196C

Commit message: Continued initial schematic capture
Parts:
- added C103, C104, C105, C107, C108, C125, C128, C135, C136, C137, C139, C140, C148, C151: 4.7 uF, azonenberg_pcb:EIA_0603_CAP_NOSILK, symbol device:C
- added C106, C111, C120, C121, C122, C123, C124, C126, C127, C129, C130, C131, C132, C133, C134, C138, C141, C142, C143, C144, C145, C146, C147, C149, C150, C152, C153, C154, C155, C156, C157: 0.47 uF, azonenberg_pcb:EIA_0402_CAP_NOSILK, symbol device:C
- added C109, C110, C112, C113, C114, C115, C116, C117, C118, C119: 0.1 uF, azonenberg_pcb:EIA_0402_CAP_NOSILK, symbol device:C
- added D10, D11, D12, D13: GREEN, azonenberg_pcb:EIA_0603_LED, symbol device:LED
- added FB10, FB11, FB12, FB7, FB8, FB9: MI0603J601R-10, azonenberg_pcb:EIA_0603_INDUCTOR_NOSILK, symbol passive-azonenberg:FERRITE_SMALL2
- added J2, J8: BEL_FUSE_0826-1G1T-23-F, azonenberg_pcb:CONN_BELFUSE_0826_1G1T_23_F, symbol special-azonenberg:BEL_FUSE_0826-1G1T-23-F
- added R100, R101, R102, R103, R104, R105, R106, R108, R109, R110, R111, R112, R113, R99: 10K, azonenberg_pcb:EIA_0402_RES_NOSILK, symbol device:R
- added R107, R114, R80, R81, R97, R98: 1K, azonenberg_pcb:EIA_0402_RES_NOSILK, symbol device:R
- added R115, R116, R82, R83, R84, R85, R86, R87, R89, R90, R91, R92, R93, R94, R96: 33, azonenberg_pcb:EIA_0402_RES_NOSILK, symbol device:R
- added R123, R124, R125, R126, R76, R77, R78, R79: 470, azonenberg_pcb:EIA_0402_RES_NOSILK, symbol device:R
- added R74, R75: 1M, azonenberg_pcb:EIA_0402_RES_NOSILK, symbol device:R
- added R88, R95: 12.1K 1%, azonenberg_pcb:EIA_0402_RES_NOSILK, symbol device:R
- added U10, U11, U12: OSC, symbol osc-azonenberg:OSC
- added U2, U9: KSZ9031RN, azonenberg_pcb:QFN_48_0.5MM_7x7MM, symbol special-azonenberg:KSZ9031RN
- U4: footprint (none) -> azonenberg_pcb:BGA_196_15x15_FULLARRAY_1MM_FTGB196
Connections:
- net FPGA_LED3: now reaches U4.A4 (IO_L2P_T0_34)
- net FPGA_LED3: now also R126.1
- net FPGA_LED0: now reaches U4.B6 (IO_0_34)
- net FPGA_LED0: now also R123.1
- net ETH3_RGMII_RX_DV: now reaches U4.C1 (IO_L11N_T1_SRCC_34)
- net ETH3_RGMII_RX_DV: now also R112.2, R93.1
- net FPGA_LED2: now reaches U4.C3 (IO_L1N_T0_34)
- net FPGA_LED2: now also R125.1
- net ETH3_RGMII_RXD0: now reaches U4.D1 (IO_L11P_T1_SRCC_34)
- net ETH3_RGMII_RXD0: now also R111.2, R92.1
- net ETH3_RGMII_RXD1: now reaches U4.D2 (IO_L10N_T1_34)
- net ETH3_RGMII_RXD1: now also R110.2, R91.1
- net FPGA_LED1: now reaches U4.D3 (IO_L1P_T0_34)
- net FPGA_LED1: now also R124.1
- net ETH3_RGMII_RXD2: now reaches U4.E2 (IO_L10P_T1_34)
- net ETH3_RGMII_RXD2: now also R109.2, R90.1
- net ETH3_MDIO: now reaches U4.F4 (IO_L12N_T1_MRCC_34)
- net ETH3_MDIO: now also U9.37 (MDIO)
- net ETH2_RGMII_RX_CLK: now reaches U4.G4 (IO_L12P_T1_MRCC_34)
- net ETH2_RGMII_RX_CLK: now also R106.2, R87.1
- net ETH3_RST_N: now reaches U4.H1 (IO_L14N_T2_SRCC_34)
- net ETH3_RST_N: now also U9.42 (RESET_N)
- net FPGA_CLK_25MHZ: now reaches U4.H2 (IO_L14P_T2_SRCC_34)
- net FPGA_CLK_25MHZ: now also R115.1
- net ETH3_MDC: now reaches U4.H3 (IO_L13N_T2_MRCC_34)
- net ETH3_MDC: now also U9.36 (MDC)
- net ETH3_RGMII_RX_CLK: now reaches U4.H4 (IO_L13P_T2_MRCC_34)
- net ETH3_RGMII_RX_CLK: now also R113.2, R94.1
- net ETH3_RGMII_TXD1: now reaches U4.J1 (IO_L15N_T2_DQS_34)
- net ETH3_RGMII_TXD1: now also U9.20 (TXD1)
- net ETH3_RGMII_TXD0: now reaches U4.J2 (IO_L15P_T2_DQS_34)
- net ETH3_RGMII_TXD0: now also U9.19 (TXD0)
- net ETH3_RGMII_TX_EN: now reaches U4.J3 (IO_L17N_T2_34)
- net ETH3_RGMII_TX_EN: now also U9.25 (TX_EN)
- net ETH3_RGMII_TX_CLK: now reaches U4.J4 (IO_L17P_T2_34)
- net ETH3_RGMII_TX_CLK: now also U9.24 (GTX_CLK)
- net ETH3_RGMII_TXD3: now reaches U4.K3 (IO_L16N_T2_34)
- net ETH3_RGMII_TXD3: now also U9.22 (TXD3)
- net ETH3_RGMII_TXD2: now reaches U4.K4 (IO_L16P_T2_34)
- net ETH3_RGMII_TXD2: now also U9.21 (TXD2)
- net ETH2_RGMII_TXD0: now reaches U4.L1 (IO_L18N_T2_34)
- net ETH2_RGMII_TXD0: now also U2.19 (TXD0)
- net ETH2_RGMII_RXD1: now reaches U4.L2 (IO_L22N_T3_34)
- net ETH2_RGMII_RXD1: now also R103.2, R84.1
- net ETH2_RGMII_RXD2: now reaches U4.L3 (IO_L22P_T3_34)
- net ETH2_RGMII_RXD2: now also R102.2, R83.1
- net ETH2_RST_N: now reaches U4.L5 (IO_25_34)
- net ETH2_RST_N: now also U2.42 (RESET_N)
- net ETH3_RGMII_RXD3: now reaches U4.M1 (IO_L18P_T2_34)
- net ETH3_RGMII_RXD3: now also R108.2, R89.1
- net ETH2_RGMII_TXD2: now reaches U4.M2 (IO_L19N_T3_VREF_34)
- net ETH2_RGMII_TXD2: now also U2.21 (TXD2)
- net ETH2_RGMII_TXD1: now reaches U4.M3 (IO_L19P_T3_34)
- net ETH2_RGMII_TXD1: now also U2.20 (TXD1)
- net ETH2_RGMII_RX_DV: now reaches U4.M4 (IO_L23N_T3_34)
- net ETH2_RGMII_RX_DV: now also R105.2, R86.1
- net ETH2_RGMII_RXD0: now reaches U4.M5 (IO_L23P_T3_34)
- net ETH2_RGMII_RXD0: now also R104.2, R85.1
- net ETH2_RGMII_TX_CLK: now reaches U4.N1 (IO_L20N_T3_34)
- net ETH2_RGMII_TX_CLK: now also U2.24 (GTX_CLK)
- net ETH2_MDIO: now reaches U4.N4 (IO_L24N_T3_34)
- net ETH2_MDIO: now also U2.37 (MDIO)
- net ETH2_RGMII_TXD3: now reaches U4.P2 (IO_L20P_T3_34)
- net ETH2_RGMII_TXD3: now also U2.22 (TXD3)
- net ETH2_RGMII_RXD3: now reaches U4.P3 (IO_L21N_T3_DQS_34)
- net ETH2_RGMII_RXD3: now also R101.2, R82.1
- net ETH2_RGMII_TX_EN: now reaches U4.P4 (IO_L21P_T3_DQS_34)
- net ETH2_RGMII_TX_EN: now also U2.25 (TX_EN)
- net ETH2_MDC: now reaches U4.P5 (IO_L24P_T3_34)
- net ETH2_MDC: now also U2.36 (MDC)
- new net: J2.16 (LED2_P), R77.2
- new net: D13.2 (A), R126.2
- new net: R95.2, U9.48 (ISET)
- new net: C118.2, J8.1 (CH3_TAP)
- new net: R99.2, U2.41 (CLK125_NDO/LED_MODE)
- new net: D12.2 (A), R125.2
- new net: R83.2, U2.28 (RXD2/MODE2)
- new net: D11.2 (A), R124.2
- new net: C117.2, J8.6 (CH2_TAP)
- new net: R100.2, U9.41 (CLK125_NDO/LED_MODE)
- new net: R92.2, U9.32 (RXD0/MODE0)
- new net: R93.2, U9.33 (RX_DV/CLK125_EN)
- new net: R82.2, U2.27 (RXD3/MODE3)
- new net: R90.2, U9.28 (RXD2/MODE2)
- new net: R96.2, U10.3 (CLK)
- new net: J2.14 (LED1_P), R76.2
- new net: R116.2, U12.3 (CLK)
- new net: R84.2, U2.31 (RXD1/MODE1)
- new net: R85.2, U2.32 (RXD0/MODE0)
- new net: R86.2, U2.33 (RX_DV/CLK125_EN)
- new net: R87.2, U2.35 (RX_CLK/PHYAD2)
- new net: R88.2, U2.48 (ISET)
- new net: C119.2, J8.7 (CH4_TAP)
- new net: C114.2, J2.1 (CH3_TAP)
- new net: D10.2 (A), R123.2
- new net: J8.14 (LED1_P), R78.2
- new net: R91.2, U9.31 (RXD1/MODE1)
- new net: R94.2, U9.35 (RX_CLK/PHYAD2)
- new net: C109.2, J2.17 (SHLD), R74.2
- new net: C116.2, J8.12 (CH1_TAP)
- new net: C110.2, J8.17 (SHLD), R75.2
- new net: C113.2, J2.6 (CH2_TAP)
- new net: C115.2, J2.7 (CH4_TAP)
- new net: R115.2, U11.3 (CLK)
- new net: R89.2, U9.27 (RXD3/MODE3)
- new net: C112.2, J2.12 (CH1_TAP)
- new net: J8.16 (LED2_P), R79.2
- new net 1V2: C105.1, C125.1, C127.1, C129.1, C131.1, C132.1, C133.1, C134.1, C137.1, C148.1, C150.1, C152.1, C154.1, C155.1, C156.1, C157.1, FB11.1, FB12.1, FB8.1, FB9.1, U2.14 (DVDDL), U2.18 (DVDDL), U2.23 (DVDDL), U2.26 (DVDDL), U2.30 (DVDDL), U2.39 (DVDDL), U9.14 (DVDDL), U9.18 (DVDDL), U9.23 (DVDDL), U9.26 (DVDDL), U9.30 (DVDDL), U9.39 (DVDDL)
- new net 1V8: R101.1, R102.1, R103.1, R108.1, R109.1, R110.1
- new net 3V3: C103.1, C104.1, C106.1, C111.1, C126.1, C135.1, C136.1, C138.1, C141.1, C147.1, C149.1, FB10.1, FB7.1, R100.1, R107.1, R114.1, R76.1, R77.1, R78.1, R79.1, R99.1, U10.1 (E/D#), U10.4 (Vdd), U11.1 (E/D#), U11.4 (Vdd), U12.1 (E/D#), U12.4 (Vdd), U2.16 (DVDDH), U2.34 (DVDDH), U2.40 (DVDDH), U9.16 (DVDDH), U9.34 (DVDDH), U9.40 (DVDDH)
- new net A3V3: C107.1, C121.1, C122.1, C124.1, C139.1, C143.1, C144.1, C146.1, FB10.2, FB7.2, U2.1 (AVDDH), U2.12 (AVDDH), U2.47 (NC/AVDDH), U9.1 (AVDDH), U9.12 (AVDDH), U9.47 (NC/AVDDH)
- new net ETH2_A1V2: C108.1, C120.1, C123.1, FB8.2, U2.4 (AVDDL), U2.9 (AVDDL)
- new net ETH2_A1V2_PLL: C128.1, C130.1, FB9.2, U2.44 (AVDDL_PLL)
- new net ETH2_A_N: J2.10 (CH1_N), U2.3 (TXRXM_A)
- new net ETH2_A_P: J2.11 (CH1_P), U2.2 (TXRXP_A)
- new net ETH2_B_N: J2.5 (CH2_N), U2.6 (TXRXM_B)
- new net ETH2_B_P: J2.4 (CH2_P), U2.5 (TXRXP_B)
- new net ETH2_CLK_25MHZ: R96.1, U2.46 (XI)
- new net ETH2_C_N: J2.2 (CH3_N), U2.8 (TXRXM_C)
- new net ETH2_C_P: J2.3 (CH3_P), U2.7 (TXRXP_C)
- new net ETH2_D_N: J2.9 (CH4_N), U2.11 (TXRXM_D)
- new net ETH2_D_P: J2.8 (CH4_P), U2.10 (TXRXP_D)
- new net ETH2_LED1_N: J2.13 (LED1_N), R97.2, U2.17 (LED1/PHYAD0)
- new net ETH2_LED2_N: J2.15 (LED2_N), R80.2, U2.15 (LED2/PHYAD1)
- new net ETH2_RGMII_MDIO: R107.2
- new net ETH3_A1V2: C140.1, C142.1, C145.1, FB11.2, U9.4 (AVDDL), U9.9 (AVDDL)
- new net ETH3_A1V2_PLL: C151.1, C153.1, FB12.2, U9.44 (AVDDL_PLL)
- new net ETH3_A_N: J8.10 (CH1_N), U9.3 (TXRXM_A)
- new net ETH3_A_P: J8.11 (CH1_P), U9.2 (TXRXP_A)
- new net ETH3_B_N: J8.5 (CH2_N), U9.6 (TXRXM_B)
- new net ETH3_B_P: J8.4 (CH2_P), U9.5 (TXRXP_B)
- new net ETH3_CLK_25MHZ: R116.1, U9.46 (XI)
- new net ETH3_C_N: J8.2 (CH3_N), U9.8 (TXRXM_C)
- new net ETH3_C_P: J8.3 (CH3_P), U9.7 (TXRXP_C)
- new net ETH3_D_N: J8.9 (CH4_N), U9.11 (TXRXM_D)
- new net ETH3_D_P: J8.8 (CH4_P), U9.10 (TXRXP_D)
- new net ETH3_LED1_N: J8.13 (LED1_N), R98.2, U9.17 (LED1/PHYAD0)
- new net ETH3_LED2_N: J8.15 (LED2_N), R81.2, U9.15 (LED2/PHYAD1)
- new net ETH3_RGMII_MDIO: R114.2
- new net GND: C103.2, C104.2, C105.2, C106.2, C107.2, C108.2, C109.1, C110.1, C111.2, C112.1, C113.1, C114.1, C115.1, C116.1, C117.1, C118.1, C119.1, C120.2, C121.2, C122.2, C123.2, C124.2, C125.2, C126.2, C127.2, C128.2, C129.2, C130.2, C131.2, C132.2, C133.2, C134.2, C135.2, C136.2, C137.2, C138.2, C139.2, C140.2, C141.2, C142.2, C143.2, C144.2, C145.2, C146.2, C147.2, C148.2, C149.2, C150.2, C151.2, C152.2, C153.2, C154.2, C155.2, C156.2, C157.2, D10.1 (K), D11.1 (K), D12.1 (K), D13.1 (K), R104.1, R105.1, R106.1, R111.1, R112.1, R113.1, R74.1, R75.1, R80.1, R81.1, R88.1, R95.1, R97.1, R98.1, U10.2 (Vss), U11.2 (Vss), U12.2 (Vss), U2.13 (NC/GND), U2.29 (VSS), U2.PAD, U9.13 (NC/GND), U9.29 (VSS), U9.PAD
- no-connect marks 0 -> 21
Other:
- note added: "Debug / GPIO LEDs"
- note added: "Strap: Disable CLK125_NDO we don't use"
- note added: "Strap: PHYADDR[2] = 0"
- note added: "Strap: PHYADR[1:0] = 2'b00"
- note added: "Strap: advertise everything but gig/half"
- note added: "Strap: dual LEDs"
- note added: "eth2 decoupling"
- note added: "eth3 decoupling"
- moved on the sheet: U4D

Commit message: Finished initial schematic, ready for signoff review
Parts:
- U10, U11, U12: value OSC -> ECS-2016MVQ-250-CN-TR; footprint (none) -> azonenberg_pcb:OSCILLATOR_2.0x1.6
Connections:
- net A3V3 renamed ETH2_A3V3
- net ETH2_A3V3: no longer C139.1, C143.1, C144.1, C146.1, FB10.2, U9.1 (AVDDH), U9.12 (AVDDH), U9.47 (NC/AVDDH)
- new net ETH3_A3V3: C139.1, C143.1, C144.1, C146.1, FB10.2, U9.1 (AVDDH), U9.12 (AVDDH), U9.47 (NC/AVDDH)
Changed lines of the file:
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@@
     (effects (font (size 1.27 1.27)) (justify left bottom))
   )
-  (label "A3V3" (at 271.78 210.82 0)
+  (label "ETH3_A3V3" (at 271.78 210.82 0)
     (effects (font (size 1.27 1.27)) (justify left bottom))
   )
@@
     (effects (font (size 1.27 1.27)) (justify right bottom))
   )
-  (label "A3V3" (at 82.55 119.38 180)
+  (label "ETH3_A3V3" (at 82.55 119.38 180)
     (effects (font (size 1.27 1.27)) (justify right bottom))
   )
@@
     (effects (font (size 1.27 1.27)) (justify left bottom))
   )
-  (label "A3V3" (at 91.44 210.82 0)
+  (label "ETH2_A3V3" (at 91.44 210.82 0)
     (effects (font (size 1.27 1.27)) (justify left bottom))
   )
@@
     (effects (font (size 1.27 1.27)) (justify left bottom))
   )
-  (label "A3V3" (at 82.55 30.48 180)
+  (label "ETH2_A3V3" (at 82.55 30.48 180)
     (effects (font (size 1.27 1.27)) (justify right bottom))
   )
@@
       (effects (font (size 1.524 1.524)))
     )
-    (property "Value" "OSC" (id 1) (at 137.795 235.4326 0)
-      (effects (font (size 1.524 1.524)))
-    )
-    (property "Footprint" "" (id 2) (at 138.43 240.03 0)
+    (property "Value" "ECS-2016MVQ-250-CN-TR" (id 1) (at 137.795 235.4326 0)
+      (effects (font (size 1.524 1.524)))
+    )
+    (property "Footprint" "azonenberg_pcb:OSCILLATOR_2.0x1.6" (id 2) (at 138.43 240.03 0)
       (effects (font (size 1.524 1.524)) hide)
     )
@@
       (effects (font (size 1.524 1.524)))
     )
-    (property "Value" "OSC" (id 1) (at 318.135 235.4326 0)
-      (effects (font (size 1.524 1.524)))
-    )
-    (property "Footprint" "" (id 2) (at 318.77 240.03 0)
+    (property "Value" "ECS-2016MVQ-250-CN-TR" (id 1) (at 318.135 235.4326 0)
+      (effects (font (size 1.524 1.524)))
+    )
+    (property "Footprint" "azonenberg_pcb:OSCILLATOR_2.0x1.6" (id 2) (at 318.77 240.03 0)
       (effects (font (size 1.524 1.524)) hide)
     )
@@
       (effects (font (size 1.524 1.524)))
     )
-    (property "Value" "OSC" (id 1) (at 306.705 86.8426 0)
-      (effects (font (size 1.524 1.524)))
-    )
-    (property "Footprint" "" (id 2) (at 307.34 91.44 0)
+    (property "Value" "ECS-2016MVQ-250-CN-TR" (id 1) (at 306.705 86.8426 0)
+      (effects (font (size 1.524 1.524)))
+    )
+    (property "Footprint" "azonenberg_pcb:OSCILLATOR_2.0x1.6" (id 2) (at 307.34 91.44 0)
       (effects (font (size 1.524 1.524)) hide)
     )
